Commit message: new urdf with asus sensor and publish echo data

File: xbot/urdf/Xbot_base.urdf (robot description, URDF)
Before this commit: robot Xbot, 13 links, 12 joints
Links:
- added link camera_platform; visual box size=0 0 0
Joints:
- added joint base_to_camera_platform: type fixed, parent base_link, child camera_platform, origin xyz=0.2 0 0.23 rpy=0 0 0, axis 0 0 1
- joint base_to_left_wheel: axis 0 1 0 -> 1 0 0
- joint base_to_right_wheel: axis 0 1 0 -> 1 0 0

Commit message: modified urdf

File: xbot/urdf/Xbot_base.urdf (robot description, URDF)
Before this commit: robot xbot, 14 links, 13 joints
Links:
- link base_link: geometry collision cylinder length=0.1 radius=0.24; visual cylinder length=0.1 radius=0.2
Joints:
- joint base_to_left_wheel: origin xyz=0 0.235 -0.0085 rpy=0 0 0 -> xyz=0 0.20 -0.0085 rpy=0 0 0; type continuous -> fixed
- joint base_to_right_wheel: origin xyz=0 -0.235 -0.0085 rpy=0 0 0 -> xyz=0 -0.20 -0.0085 rpy=0 0 0; type continuous -> fixed

Commit message: add debug_sensors_publisher

File: xbot/urdf/Xbot_base.urdf (robot description, URDF)
Before this commit: robot xbot, 14 links, 13 joints
Joints:
- joint base_to_camera_platform: origin xyz=0.2 0 0.23 rpy=0 0 0 -> xyz=0.078 0 0.23 rpy=0 0 0

Commit message: new safety control

File: xbot/urdf/Xbot_base.urdf (robot description, URDF)
Before this commit: robot xbot, 14 links, 13 joints
Joints:
- joint base_to_camera_platform: origin xyz=0.078 0 0.23 rpy=0 0 0 -> xyz=0.2 0 0.23 rpy=0 0 0
