Commit message: new

File: xbot_bringup/urdf/Xbot.urdf.xacro (robot description, xacro)
@@ -6,5 +6,5 @@
 -->
 <robot name="xbot" xmlns:xacro="http://ros.org/wiki/xacro">
-  <xacro:include filename="./Xbot_base_rplidar_asus.urdf" />
+  <xacro:include filename="./Xbot_base_rplidar.urdf" />
   <xbot/>
   <sensor_asus_xtion_pro          parent="camera_platform"/>

File: xbot_bringup/urdf/Xbot_base_rplidar.urdf (robot description, URDF)
Before this commit: robot xbot, 15 links, 14 joints
Links:
- added link global_scan
- link platform1: geometry collision box size=.14 .14 1.1; visual box size=.12 .12 .77
- link platform2: geometry visual cylinder length=0.85 radius=0.055
- link platform3: geometry visual cylinder length=0.12 radius=0.055
Joints:
- removed joint base_to_camera_platform
- added joint laser_to_global_scan: type fixed, parent laser, child global_scan, origin xyz=0 0 0.3 rpy=0 0 0, axis 1 0 0
- added joint platform1_to_camera_platform: type fixed, parent platform1, child camera_platform, origin xyz=0.09 0 0.20 rpy=0 0 0, axis 0 0 1
- joint base_to_frontleft_omniwheel: origin xyz=0.2 0.1 -0.07 rpy=0 0 0 -> xyz=0.2 0.1 0.005 rpy=0 0 0
- joint base_to_frontright_omniwheel: origin xyz=0.2 -0.1 -0.07 rpy=0 0 0 -> xyz=0.2 -0.1 0.005 rpy=0 0 0
- joint base_to_laser: origin xyz=0.14 0 0.06 rpy=0 0 0 -> xyz=0.14 0 0.135 rpy=0 0 0
- joint base_to_left_wheel: origin xyz=0 0.20 -0.0085 rpy=0 0 0 -> xyz=0 0.20 0.075 rpy=0 0 0
- joint base_to_platform1: origin xyz=0 0 0.4 rpy=0 0 0 -> xyz=0 0 0.475 rpy=0 0 0
- joint base_to_rearleft_omniwheel: origin xyz=-0.2 .1 -0.07 rpy=0 0 0 -> xyz=-0.2 .1 0.005 rpy=0 0 0
- joint base_to_rearright_omniwheel: origin xyz=-0.2 -0.1 -0.07 rpy=0 0 0 -> xyz=-0.2 -0.1 0.005 rpy=0 0 0
- joint base_to_right_wheel: origin xyz=0 -0.20 -0.0085 rpy=0 0 0 -> xyz=0 -0.20 0.075 rpy=0 0 0
- joint platform1_to_platform2: type prismatic -> fixed
- joint platform2_to_platform3: type revolute -> fixed
- joint platform4_to_platform5: type revolute -> fixed

File: xbot_bringup/urdf/asus_xtion_pro.urdf.xacro (robot description, xacro)
@@ -1,6 +1,5 @@
 <?xml version="1.0"?>
 <robot name="sensor_asus_xtion_pro" xmlns:xacro="http://ros.org/wiki/xacro">
-  <xacro:include filename="$(find turtlebot_description)/urdf/turtlebot_gazebo.urdf.xacro"/>
-  <xacro:include filename="$(find turtlebot_description)/urdf/turtlebot_properties.urdf.xacro"/>
+  <xacro:include filename="$(find xbot_bringup)/urdf/common_properties.urdf.xacro"/>
   <!-- Xacro properties -->
   <xacro:property name="M_SCALE" value="0.001"/>
@@ -8,4 +7,9 @@
   <xacro:property name="asus_xtion_pro_depth_rel_rgb_py" value="0.0270" />
   <xacro:property name="asus_xtion_pro_cam_rel_rgb_py"   value="-0.0220" />
+  <xacro:property name="cam_px" value="0" />
+  <xacro:property name="cam_pz" value="0" />
+  <xacro:property name="cam_or" value="0" />
+  <xacro:property name="cam_op" value="0" />
+  <xacro:property name="cam_oy" value="0" />
   <!-- Parameterised in part by the values in turtlebot_properties.urdf.xacro -->
   <xacro:macro name="sensor_asus_xtion_pro" params="parent">
@@ -33,5 +37,5 @@
         <origin xyz="-0.015 0.0035 0.004" rpy="0 0 0"/>
         <geometry>
-          <mesh filename="package://turtlebot_description/meshes/sensors/xtion_pro_camera.dae"/>
+          <mesh filename="package://xbot_bringup/meshes/sensors/xtion_pro_camera.dae"/>
         </geometry>
       </visual>
@@ -66,5 +70,5 @@
     <!-- Asus mount -->
     <joint name="mount_asus_xtion_pro_joint" type="fixed">
-      <origin xyz="-0.1024 0.0 0.272" rpy="0 0 0"/>
+      <origin xyz="-0.02 0.0 -0.03" rpy="0 0 0"/>
       <parent link="${parent}"/>
       <child link="mount_asus_xtion_pro_link"/>
@@ -74,5 +78,5 @@
         <origin xyz="0 0 0" rpy="${-M_PI/2} 0 0"/>
         <geometry>
-          <mesh filename="package://turtlebot_description/meshes/sensors/xtion_pro_stack.dae"/>
+          <mesh filename="package://xbot_bringup/meshes/sensors/xtion_pro_stack.dae"/>
         </geometry>
       </visual>
