Commit message: new

File: xbot_bringup/urdf/Xbot_base_rplidar.urdf (robot description, URDF)
Before this commit: robot xbot, 15 links, 14 joints
Links:
- removed link rplidar
- added link laser; visual cylinder length=0.045 radius=0.045
Joints:
- removed joint base_to_rplidar
- added joint base_to_laser: type fixed, parent base_link, child laser, origin xyz=0.14 0 0.06 rpy=0 0 0, axis 1 0 0

Commit message: new

File: xbot_bringup/urdf/Xbot_base_rplidar.urdf (robot description, URDF)
Before this commit: robot xbot, 16 links, 15 joints
Joints:
- removed joint laser_to_global_scan
- added joint base_link_to_global_scan: type fixed, parent base_link, child global_scan, origin xyz=0.14 0 0.435 rpy=0 0 0, axis 1 0 0
- joint base_to_laser: origin xyz=0.14 0 0.135 rpy=0 0 0 -> xyz=0.15 0 0.135 rpy=0 0 0
- joint platform1_to_camera_platform: origin xyz=0.09 0 0.20 rpy=0 0 0 -> xyz=0.10 0 0.20 rpy=0 0 0

Commit message: 1.delete scan180  2.modify rplidar location

File: xbot_bringup/urdf/Xbot_base_rplidar.urdf (robot description, URDF)
Before this commit: robot xbot, 16 links, 15 joints
Joints:
- joint base_to_laser: origin xyz=0.15 0 0.135 rpy=0 0 0 -> xyz=0 0 0.17 rpy=0 0 3.1416
